Commit message: Add files via upload

File: ur_ros_cartesian_control/ur_ros_cartesian_control/urdf/manufacture_system.xacro (robot description, xacro)
@@ -61,5 +61,5 @@
             prefix="ur_"
             />
-        <link name="tool_holder_link">
+        <link name="ur_tool_holder_link">
             <visual>
                 <origin xyz="-0.0315 0.078 0" rpy="1.57079632679 0 0"/>
@@ -81,5 +81,5 @@
             </inertial>
         </link>
-        <link name="ee_link">
+        <link name="ur_ee_link">
             <visual>
                 <origin xyz="-0.01 -0.1075 -0.055" rpy="-1.047200654 0 0"/>
@@ -103,7 +103,7 @@
         <link name="object_zig_link">
             <visual>
-                <origin xyz="-0.11 -0.11 0" rpy="0 0 0"/>
+                <origin xyz="-0.0975 -0.0975 0" rpy="0 0 0"/>
                 <geometry>
-                    <mesh filename="package://ur_ros_cartesian_control/meshes/grinding_test_zig.STL" scale="0.001 0.001 0.001"/>
+                    <mesh filename="package://ur_ros_cartesian_control/meshes/grinding_demo_zig.STL" scale="0.001 0.001 0.001"/>
                 </geometry>
             </visual>
@@ -125,5 +125,5 @@
                 <origin xyz="-0.05 -0.05 0" rpy="0 0 0"/>
                 <geometry>
-                    <mesh filename="package://ur_ros_cartesian_control/meshes/grinding_test.STL" scale="0.001 0.001 0.001"/>
+                    <mesh filename="package://ur_ros_cartesian_control/meshes/grinding_test_2.STL" scale="0.001 0.001 0.001"/>
                 </geometry>
             </visual>
@@ -158,21 +158,21 @@
         <joint name="flange_to_holder" type="fixed">
             <parent link="ur_tool0"/>
-            <child link="tool_holder_link"/>
+            <child link="ur_tool_holder_link"/>
             <origin xyz="0 0 0" rpy="0 0 0"/>
         </joint>
         <joint name="holder_to_ee" type="fixed">
-            <parent link="tool_holder_link"/>
-            <child link="ee_link"/>
-            <origin xyz="0 0.065 0.115" rpy="0 0 0"/>
+            <parent link="ur_tool_holder_link"/>
+            <child link="ur_ee_link"/>
+            <origin xyz="0 0.065 0.117" rpy="0 0 0"/>
         </joint>
         <joint name="table_to_zig" type="fixed">
             <parent link="table_base_link"/>
             <child link="object_zig_link"/>
-            <origin xyz="-0.0125 -0.2 ${base_height}" rpy="0 0 0"/>
+            <origin xyz="0 -0.28725 ${base_height}" rpy="0 0 0"/>
         </joint>
         <joint name="zig_to_object" type="fixed">
             <parent link="object_zig_link"/>
             <child link="object_base_link"/>
-            <origin xyz="0 0 0.1" rpy="0 0 0"/>
+            <origin xyz="0 0 0.07" rpy="0 0 0"/>
         </joint>
     </xacro:macro>
